File: robot_elshema/robot_elshema.sch (KiCad schematic (older format))
At the start: 17 parts, among them M1 motor, M2 motor

Commit message: Update el. sheme
Parts:
- removed MUX1: CD4051BE, symbol CD4051BE
- removed SC1, SC2, SC3, SC4, SC5, SC6, SC7, SC8: QRE1113, symbol QRE1113
- added BAT1: Baterija, symbol Battery
- added BT1: RN-42, symbol RN-42
- added C3: 22uF, symbol CP1_Small
- added D1: GREEN, symbol LED
- added D2: RED, symbol LED
- added MUX1: CD4051BM96, robot:CD4051, symbol CD4051BM96
- added Q1: Q_NPN_CBE, symbol Q_NPN_CBE
- added Q2: Q_PMOS_GSD, symbol Q_PMOS_GSD
- added R10, R11, R12, R13, R14, R15, R16, R17, R3, R4, R5, R6: 10K, symbol R
- added R7: 1K, symbol R
- added R8, R9: 330, symbol R
- added SC1, SC2, SC3, SC4, SC5, SC6, SC7, SC8: QRE1113GR, symbol QRE1113GR
- added SW1: SW_PUSH, symbol SW_PUSH
- added SW2: SWITCH, symbol SWITCH
- added VLT1: TXB0108, symbol TXB0108
Connections:
- net labels added: +9VA, 1, 13.3.2017, AR3.3, ARRX, ARTX, BTRX, BTTX, BUT, ENCDA, ENCDB, ENCLA, ENCLB, MD1, MD2, ML1, ML2, MUX, MUXA, MUXB, MUXC, SC1, SC2, SC3, SC4, SC5, SC6, SC7, SC8, SCON, Shema robota za sledenje črti, VBAT
- wire segments 165 -> 227
- no-connect marks 0 -> 12
Other:
- note added: "BLUETOOTH"
- note added: "MIKROKRMILNIK"
- note added: "MOTORJA IN ENKODERJA"
- note added: "MULTIPLEKSER"
- note added: "NAPAJANJE"
- note added: "PRETVORNIK NAPETOSTI"
- note added: "SENZORJI ČRT"
- note added: "TIPKA"
- moved on the sheet: C1, C2, Hmostic1, M1, M2, R1, R2, UC1

Commit message: Posodobljena el. shema in dodan PCB robota
Parts:
- removed Q1: Q_NPN_CBE, symbol Q_NPN_CBE
- removed Q2: Q_PMOS_GSD, symbol Q_PMOS_GSD
- removed UC1: Arduino_Micro, symbol Arduino_Micro
- removed VLT1: TXB0108, symbol TXB0108
- added Q?: BC237, TO_SOT_Packages_THT:TO-92_Molded_Narrow, symbol BC237
- added Q?: TP0610T, TO_SOT_Packages_SMD:SOT-23, symbol TP0610T
- added R14: 10K, Resistors_SMD:R_0805_HandSoldering, symbol R
- added U?: ARDUINO_MICRO_SHIELD, arduino_micro_shield:ARDUINO_MICRO_SHIELD, symbol ARDUINO_MICRO_SHIELD
- added VLT1: TXB0102, TXB0102:SOP-08, symbol TXB0102
- BAT1: footprint (none) -> robot:batteryholder
- BT1: footprint (none) -> robot:RN-42
- C1: footprint (none) -> Capacitors_SMD:C_0805_HandSoldering
- C2: renamed from C3; footprint (none) -> Capacitors_SMD:C_0805_HandSoldering
- C3: renamed from C2; footprint (none) -> Capacitors_SMD:C_0805_HandSoldering
- D1, D2: footprint (none) -> LEDs:LED_0805
- Hmostic1: footprint (none) -> L293D:DIL16
- M1, M2: footprint (none) -> robot:Motor
- R1, R10, R11, R12, R13, R8, R9: footprint (none) -> Resistors_SMD:R_0805_HandSoldering
- R15: renamed from R14; footprint (none) -> Resistors_SMD:R_0805_HandSoldering
- R16: renamed from R15; footprint (none) -> Resistors_SMD:R_0805_HandSoldering
- R17: renamed from R16; footprint (none) -> Resistors_SMD:R_0805_HandSoldering
- R18: renamed from R17; footprint (none) -> Resistors_SMD:R_0805_HandSoldering
- R2: renamed from R3; footprint (none) -> Resistors_SMD:R_0805_HandSoldering
- R3: renamed from R4; footprint (none) -> Resistors_SMD:R_0805_HandSoldering
- R4: renamed from R5; footprint (none) -> Resistors_SMD:R_0805_HandSoldering
- R5: renamed from R6; footprint (none) -> Resistors_SMD:R_0805_HandSoldering
- R6: renamed from R7; footprint (none) -> Resistors_SMD:R_0805_HandSoldering
- R7: renamed from R2; footprint (none) -> Resistors_SMD:R_0805_HandSoldering
- SC1, SC2, SC3, SC4, SC5, SC6, SC7, SC8: footprint (none) -> robot:QRE1113GR
- SW1: footprint (none) -> robot:SW_SPST_B3U-3000P-B
- SW2: footprint (none) -> robot:SW_SPST_B3U-3100P-B
Connections:
- net labels added: 2
- net labels removed: 1
- wire segments 227 -> 232
- no-connect marks 12 -> 26
